Commit message: Added Sensors

File: catkin_ws/src/hector_quadrotor/hector_quadrotor_description/urdf/quadrotor_base.urdf.xacro (robot description, xacro)
@@ -7,5 +7,5 @@
     <link name="base_link">
       <inertial>
-        <mass value="1.477" />
+        <mass value="3.8" />
         <origin xyz="0 0 0" />
         <inertia ixx="0.01152" ixy="0.0" ixz="0.0" iyy="0.01152" iyz="0.0" izz="0.0218" />
@@ -25,6 +25,14 @@
     </link>
     <!-- Sonar height sensor -->
-    <xacro:sonar_sensor name="sonar" parent="base_link" ros_topic="sonar_height" update_rate="10" min_range="0.03" max_range="3.0" field_of_view="${40*pi/180}" ray_count="3">
+    <xacro:sonar_sensor name="sonar" parent="base_link" ros_topic="sonar_height" update_rate="10" min_range="0.1" max_range="5.0" field_of_view="${60*pi/180}" ray_count="2">
       <origin xyz="-0.16 0.0 -0.012" rpy="0 ${90*pi/180} 0"/>
+    </xacro:sonar_sensor>
+    <!-- Infrared upward sensor -->
+    <xacro:sonar_sensor name="infrared_narrow" parent="base_link" ros_topic="upward_infrared_narrow" update_rate="10" min_range="0.01" max_range="5.0" field_of_view="${3*pi/180}" ray_count="1">
+      <origin xyz="0.07 0.0 0.04" rpy="0 ${-90*pi/180} 0"/>
+    </xacro:sonar_sensor>
+    <!-- Infrared upward sensor -->
+    <xacro:sonar_sensor name="infrared_wide" parent="base_link" ros_topic="upward_infrared_wide" update_rate="10" min_range="0.01" max_range="5.0" field_of_view="${10*pi/180}" ray_count="1">
+      <origin xyz="0.05 0.0 0.04" rpy="0 ${-90*pi/180} 0"/>
     </xacro:sonar_sensor>
   </xacro:macro>

Commit message: Updated Mass in Line 12
1.4 is close to the original value and works with the provided controller.

File: catkin_ws/src/hector_quadrotor/hector_quadrotor_description/urdf/quadrotor_base.urdf.xacro (robot description, xacro)
@@ -7,5 +7,5 @@
     <link name="base_link">
       <inertial>
-        <mass value="3.8" />
+        <mass value="1.4" />
         <origin xyz="0 0 0" />
         <inertia ixx="0.01152" ixy="0.0" ixz="0.0" iyy="0.01152" iyz="0.0" izz="0.0218" />

Commit message: Added Zero Mass Payloads to the Model

File: catkin_ws/src/hector_quadrotor/hector_quadrotor_description/urdf/quadrotor_base.urdf.xacro (robot description, xacro)
@@ -3,4 +3,5 @@
   <xacro:include filename="$(find hector_sensors_description)/urdf/sonar_sensor.urdf.xacro" />
   <xacro:property name="pi" value="3.1415926535897931" />
+  <xacro:property name="size" value="0.022" />
   <!-- Main quadrotor link -->
   <xacro:macro name="quadrotor_base_macro">
@@ -24,4 +25,52 @@
       </collision>
     </link>
+    <link name="left_payload">
+      <inertial>
+        <mass value="0.0" />
+        <origin xyz="0 0 0" />
+        <inertia ixx="0.0" ixy="0.0" ixz="0.0" iyy="0.0" iyz="0.0" izz="0.0" />
+      </inertial>
+      <visual>
+        <origin xyz="0 0 0" rpy="0 0 -${pi/2}" />
+        <geometry>
+          <mesh filename="package://hector_quadrotor_description/meshes/assembly/Payload_Assembly.stl" scale= "${size} ${size} ${size}"/>
+        </geometry>
+      </visual>
+      <collision>
+        <origin xyz="0 0 0" rpy="0 0 -${pi/2}" />
+        <geometry>
+          <mesh filename="package://hector_quadrotor_description/meshes/assembly/Payload_Assembly.stl" scale= "${size} ${size} ${size}"/>
+        </geometry>
+      </collision>
+    </link>
+    <link name="right_payload">
+      <inertial>
+        <mass value="0.0" />
+        <origin xyz="0 0 0" />
+        <inertia ixx="0.0" ixy="0.0" ixz="0.0" iyy="0.0" iyz="0.0" izz="0.0" />
+      </inertial>
+      <visual>
+        <origin xyz="0 0 0" rpy="0 0 ${pi/2}" />
+        <geometry>
+          <mesh filename="package://hector_quadrotor_description/meshes/assembly/Payload_Assembly.stl" scale= "${size} ${size} ${size}"/>
+        </geometry>
+      </visual>
+      <collision>
+        <origin xyz="0 0 0" rpy="0 0 ${pi/2}" />
+        <geometry>
+          <mesh filename="package://hector_quadrotor_description/meshes/assembly/Payload_Assembly.stl" scale= "${size} ${size} ${size}"/>
+        </geometry>
+      </collision>
+    </link>
+    <joint name="base_to_right_payload" type="fixed">
+      <parent link="base_link"/>
+      <child link="right_payload"/>
+      <origin xyz="-0.05 -0.035 -0.13" />
+    </joint>
+    <joint name="base_to_left_payload" type="fixed">
+      <parent link="base_link"/>
+      <child link="left_payload"/>
+      <origin xyz="0.02 0.035 -0.13" />
+    </joint>
     <!-- Sonar height sensor -->
     <xacro:sonar_sensor name="sonar" parent="base_link" ros_topic="sonar_height" update_rate="10" min_range="0.1" max_range="5.0" field_of_view="${60*pi/180}" ray_count="2">

File: catkin_ws/src/hector_quadrotor/hector_quadrotor_description/urdf/quadrotor_dji_m200.urdf.xacro (robot description, xacro)
@@ -11,9 +11,4 @@
       <origin xyz="0.0 0.0 -0.08" rpy="0 ${M_PI/2} 0"/>
     </xacro:generic_camera>
-    <!-- Forward facing camera
-    <xacro:include filename="$(find hector_sensors_description)/urdf/generic_stereo_camera.urdf.xacro" />
-    <xacro:generic_stereo_camera name="front_cam" parent="base_link" ros_topic="camera/image_f" cam_info_topic="camera/camera_info_f" update_rate="20" res_x="640" res_y="480" image_format="BAYER_RGGB8" hfov="60" baseline="0.166">
-      <origin xyz="0.05 0.083 -0.06" rpy="0 0 0"/>
-    </xacro:generic_stereo_camera> -->
     <!-- Forward Facing Camera -->
     <xacro:include filename="$(find hector_quadrotor_description)/urdf/kinect_camera.urdf.xacro" />

Commit message: Costmap Clears Correctly, Payload Commented out (Performance Issue)

File: catkin_ws/src/hector_quadrotor/hector_quadrotor_description/urdf/quadrotor_base.urdf.xacro (robot description, xacro)
@@ -25,4 +25,5 @@
       </collision>
     </link>
+    <!-- Payload Links
     <link name="left_payload">
       <inertial>
@@ -72,5 +73,5 @@
       <child link="left_payload"/>
       <origin xyz="0.02 0.035 -0.13" />
-    </joint>
+    </joint> -->
     <!-- Sonar height sensor -->
     <xacro:sonar_sensor name="sonar" parent="base_link" ros_topic="sonar_height" update_rate="10" min_range="0.1" max_range="5.0" field_of_view="${60*pi/180}" ray_count="2">

Commit message: Added Recording Feature to Landing Node

File: catkin_ws/src/hector_quadrotor/hector_quadrotor_description/urdf/quadrotor_base.urdf.xacro (robot description, xacro)
@@ -25,5 +25,5 @@
       </collision>
     </link>
-    <!-- Payload Links
+    <!-- Payload Links -->
     <link name="left_payload">
       <inertial>
@@ -73,5 +73,5 @@
       <child link="left_payload"/>
       <origin xyz="0.02 0.035 -0.13" />
-    </joint> -->
+    </joint>
     <!-- Sonar height sensor -->
     <xacro:sonar_sensor name="sonar" parent="base_link" ros_topic="sonar_height" update_rate="10" min_range="0.1" max_range="5.0" field_of_view="${60*pi/180}" ray_count="2">
